File: hw/BodyTempUnit-e7.sch (KiCad schematic (older format))
At the start: 27 parts, among them IC1 MAX481CUA, IC2 MEGA8-MI, U1 MAX30205MTA+21-0137I_T833-2-M, U2 LSM6DS3, U3 MCP1801T-3302I_OT

Commit message: some rerouting
Parts:
- removed COM_IN1, COM_OUT1: 53?-05261, BodyTempUnit-e7:53261-05, symbol BodyTempUnit-e7-eagle-import:53?-05261
- added J1: CONN_IN, Connector_Molex:Molex_PicoBlade_53261-0571_1x05-1MP_P1.25mm_Horizontal, symbol Connector_Generic:Conn_01x05
- added J2: CONN_OUT, Connector_Molex:Molex_PicoBlade_53261-0571_1x05-1MP_P1.25mm_Horizontal, symbol Connector_Generic:Conn_01x05
Connections:
- net GND: no longer U1.5 (A2), U1.6 (A1), U1.7 (A0)
- net RS485_+: now also J1.2 (Pin_2), J2.4 (Pin_4)
- net RS485_-: now also J1.3 (Pin_3), J2.3 (Pin_3)
- net SIG_IN: now also J1.4 (Pin_4)
- net SIG_OUT: now also IC2.10 (PD6(AIN0)), J2.2 (Pin_2); no longer IC2.12 (PB0(ICP))
- net VIN: now also J1.5 (Pin_5), J2.1 (Pin_1)
- net at R12.1: now also IC2.12 (PB0(ICP)); no longer IC2.11 (PD7(AIN1))
- new net: J1.1 (Pin_1), J2.5 (Pin_5)
- new net: U1.5 (A2), U1.6 (A1), U1.7 (A0)
Changed lines of the file:
@@
 Wire Wire Line
 	8000 1000 8000 900
-Connection ~ 8000 900
 Text Label 8400 900  0    10   ~ 0
 VCC
@@
 VCC
 Wire Wire Line
-	1900 1800 2100 1800
-Text Label 2100 1800 0    50   ~ 0
-SIG_IN
-Wire Wire Line
 	4300 4600 4500 4600
 Text Label 4500 4600 0    50   ~ 0
@@
 Wire Wire Line
 	9800 3400 9800 3700
-Wire Wire Line
-	9700 2900 9800 2900
-Wire Wire Line
-	9800 2900 9800 3000
-Wire Wire Line
-	9800 3000 9800 3100
-Wire Wire Line
-	9800 3100 9800 3400
-Wire Wire Line
-	9700 3000 9800 3000
-Wire Wire Line
-	9700 3100 9800 3100
-Connection ~ 9800 3400
-Connection ~ 9800 3000
-Connection ~ 9800 3100
 Text Label 9700 3400 0    10   ~ 0
 GND
@@
 Text Label 6000 4900 0    10   ~ 0
 GND
-Wire Wire Line
-	1900 1600 2100 1600
-Text Label 2100 1600 0    50   ~ 0
+Text Label 1600 1600 0    50   ~ 0
 RS485_+
-Text Label 2100 1100 0    50   ~ 0
+Text Label 1600 1100 0    50   ~ 0
 RS485_+
-Wire Wire Line
-	1900 1700 2100 1700
-Text Label 2100 1700 0    50   ~ 0
+Text Label 1600 1700 0    50   ~ 0
 RS485_-
-Text Label 2100 1000 0    50   ~ 0
+Text Label 1600 1000 0    50   ~ 0
 RS485_-
 Wire Wire Line
@@
 Text Label 4500 4400 0    50   ~ 0
 RS485_RO
-Wire Wire Line
-	1900 900  2100 900
-Text Label 2100 900  0    50   ~ 0
-SIG_OUT
-Text Label 2100 900  0    50   ~ 0
-SIG_OUT
-Wire Wire Line
-	4300 5300 4500 5300
-Text Label 4500 5300 0    50   ~ 0
-SIG_OUT
 Wire Wire Line
 	4300 3900 4800 3900
@@
 Wire Wire Line
 	5100 5300 5200 5300
-$Comp
-L BodyTempUnit-e7-eagle-import:MAX30205MTA+21-0137I_T833-2-M U1
-U 1 1 94FABF20
-P 8200 2900
-F 0 "U1" H 8814 3359 69  0000 L BNN
-F 1 "MAX30205MTA+21-0137I_T833-2-M" H 8789 3259 69  0000 L BNN
-F 2 "BodyTempUnit-e7:21-0137I_T833-2-M" H 8200 2900 50  0001 C CNN
-F 3 "" H 8200 2900 50  0001 C CNN
-	1    8200 2900
-	1    0    0    -1
-$EndComp
-$Comp
-L BodyTempUnit-e7-eagle-import:53?-05261 COM_IN1
-U 1 1 530F4A61
-P 1800 1900
-F 0 "COM_IN1" H 1900 1870 51  0000 L BNN
-F 1 "53?-05261" H 1770 1955 59  0001 L BNN
-F 2 "BodyTempUnit-e7:53261-05" H 1800 1900 50  0001 C CNN
-F 3 "" H 1800 1900 50  0001 C CNN
-	1    1800 1900
-	-1   0    0    1
-$EndComp
-$Comp
-L BodyTempUnit-e7-eagle-import:53?-05261 COM_IN1
-U 2 1 530F4A6D
-P 1800 1800
-F 0 "COM_IN1" H 1900 1770 51  0000 L BNN
-F 1 "53?-05261" H 1770 1855 59  0001 L BNN
-F 2 "BodyTempUnit-e7:53261-05" H 1800 1800 50  0001 C CNN
-F 3 "" H 1800 1800 50  0001 C CNN
-	2    1800 1800
-	-1   0    0    1
-$EndComp
-$Comp
-L BodyTempUnit-e7-eagle-import:53?-05261 COM_IN1
-U 3 1 530F4A69
-P 1800 1700
-F 0 "COM_IN1" H 1900 1670 51  0000 L BNN
-F 1 "53?-05261" H 1770 1755 59  0001 L BNN
-F 2 "BodyTempUnit-e7:53261-05" H 1800 1700 50  0001 C CNN
-F 3 "" H 1800 1700 50  0001 C CNN
-	3    1800 1700
-	-1   0    0    1
-$EndComp
-$Comp
-L BodyTempUnit-e7-eagle-import:53?-05261 COM_IN1
-U 4 1 530F4A75
-P 1800 1600
-F 0 "COM_IN1" H 1900 1570 51  0000 L BNN
-F 1 "53?-05261" H 1770 1655 59  0001 L BNN
-F 2 "BodyTempUnit-e7:53261-05" H 1800 1600 50  0001 C CNN
-F 3 "" H 1800 1600 50  0001 C CNN
-	4    1800 1600
-	-1   0    0    1
-$EndComp
-$Comp
-L BodyTempUnit-e7-eagle-import:53?-05261 COM_IN1
-U 5 1 530F4A71
-P 1800 1500
-F 0 "COM_IN1" H 1900 1470 51  0000 L BNN
-F 1 "53?-05261" H 1770 1555 59  0001 L BNN
-F 2 "BodyTempUnit-e7:53261-05" H 1800 1500 50  0001 C CNN
-F 3 "" H 1800 1500 50  0001 C CNN
-	5    1800 1500
-	-1   0    0    1
-$EndComp
-$Comp
-L BodyTempUnit-e7-eagle-import:53?-05261 COM_OUT1
-U 1 1 ACCF8423
-P 1800 1200
-F 0 "COM_OUT1" H 1900 1170 51  0000 L BNN
-F 1 "53?-05261" H 1770 1255 59  0001 L BNN
-F 2 "BodyTempUnit-e7:53261-05" H 1800 1200 50  0001 C CNN
-F 3 "" H 1800 1200 50  0001 C CNN
-	1    1800 1200
-	-1   0    0    1
-$EndComp
-$Comp
-L BodyTempUnit-e7-eagle-import:53?-05261 COM_OUT1
-U 2 1 ACCF842F
-P 1800 1100
-F 0 "COM_OUT1" H 1900 1070 51  0000 L BNN
-F 1 "53?-05261" H 1770 1155 59  0001 L BNN
-F 2 "BodyTempUnit-e7:53261-05" H 1800 1100 50  0001 C CNN
-F 3 "" H 1800 1100 50  0001 C CNN
-	2    1800 1100
-	-1   0    0    1
-$EndComp
-$Comp
-L BodyTempUnit-e7-eagle-import:53?-05261 COM_OUT1
-U 3 1 ACCF842B
-P 1800 1000
-F 0 "COM_OUT1" H 1900 970 51  0000 L BNN
-F 1 "53?-05261" H 1770 1055 59  0001 L BNN
-F 2 "BodyTempUnit-e7:53261-05" H 1800 1000 50  0001 C CNN
-F 3 "" H 1800 1000 50  0001 C CNN
-	3    1800 1000
-	-1   0    0    1
-$EndComp
-$Comp
-L BodyTempUnit-e7-eagle-import:53?-05261 COM_OUT1
-U 4 1 ACCF8437
-P 1800 900
-F 0 "COM_OUT1" H 1900 870 51  0000 L BNN
-F 1 "53?-05261" H 1770 955 59  0001 L BNN
-F 2 "BodyTempUnit-e7:53261-05" H 1800 900 50  0001 C CNN
-F 3 "" H 1800 900 50  0001 C CNN
-	4    1800 900
-	-1   0    0    1
-$EndComp
-$Comp
-L BodyTempUnit-e7-eagle-import:53?-05261 COM_OUT1
-U 5 1 ACCF8433
-P 1800 800
-F 0 "COM_OUT1" H 1900 770 51  0000 L BNN
-F 1 "53?-05261" H 1770 855 59  0001 L BNN
-F 2 "BodyTempUnit-e7:53261-05" H 1800 800 50  0001 C CNN
-F 3 "" H 1800 800 50  0001 C CNN
-	5    1800 800
-	-1   0    0    1
-$EndComp
 $Comp
 L BodyTempUnit-e7-eagle-import:LSM6DS3 U2
@@
 $EndComp
 $Comp
-L BodyTempUnit-e7-eagle-import:VCC #SUPPLY06
-U 1 1 A7CD5EB6
-P 8000 2400
-F 0 "#SUPPLY06" H 8000 2400 50  0001 C CNN
-F 1 "VCC" H 7960 2540 59  0000 L BNN
-F 2 "" H 8000 2400 50  0001 C CNN
-F 3 "" H 8000 2400 50  0001 C CNN
-	1    8000 2400
-	1    0    0    -1
-$EndComp
-$Comp
 L BodyTempUnit-e7-eagle-import:GND #GND05
 U 1 1 5B6A58CA
@@
 	1    0    0    -1
 $EndComp
-Wire Wire Line
-	1900 1000 2100 1000
-Wire Wire Line
-	1900 1100 2100 1100
 Wire Wire Line
 	6850 1050 7150 1050
@@
 	5100 5400 4300 5400
 Wire Wire Line
-	5100 5100 4300 5100
-Wire Wire Line
 	5100 5100 5100 4900
 Wire Wire Line
@@
 Text Label 4500 4900 0    50   ~ 0
 RS485_DE
-NoConn ~ 4300 5000
 $Comp
 L power:PWR_FLAG #FLG0101
@@
 Wire Wire Line
 	2750 7250 2750 7300
-Wire Wire Line
-	1900 1200 2050 1200
-Wire Wire Line
-	2050 1500 1900 1500
 $Comp
 L BodyTempUnit-e7-eagle-import:GND #GND0105
 U 1 1 5CFD39BA
-P 2200 1350
-F 0 "#GND0105" H 2200 1350 50  0001 C CNN
-F 1 "GND" H 2100 1250 59  0000 L BNN
-F 2 "" H 2200 1350 50  0001 C CNN
-F 3 "" H 2200 1350 50  0001 C CNN
-	1    2200 1350
-	1    0    0    -1
-$EndComp
-Wire Wire Line
-	2050 1200 2050 1500
-Wire Wire Line
-	2050 1200 2200 1200
-Wire Wire Line
-	2200 1200 2200 1250
-Connection ~ 2050 1200
-Wire Wire Line
-	1900 800  1950 800
+P 1500 2200
+F 0 "#GND0105" H 1500 2200 50  0001 C CNN
+F 1 "GND" H 1400 2100 59  0000 L BNN
+F 2 "" H 1500 2200 50  0001 C CNN
+F 3 "" H 1500 2200 50  0001 C CNN
+	1    1500 2200
+	1    0    0    -1
+$EndComp
 Wire Wire Line
 	2700 800  2700 1200
 Connection ~ 2700 1200
 Wire Wire Line
-	1900 1900 1950 1900
-Wire Wire Line
-	1950 1900 1950 800
-Connection ~ 1950 800
-Wire Wire Line
-	1950 800  2700 800
+	2150 1900 2150 800
+Connection ~ 2150 800
+Wire Wire Line
+	2150 800  2700 800
 Text Label 2700 800  0    50   ~ 0
 VIN
+$Comp
+L BodyTempUnit-e7-eagle-import:MAX30205MTA+21-0137I_T833-2-M U1
+U 1 1 94FABF20
+P 8200 2900
+F 0 "U1" H 8814 3359 69  0000 L BNN
+F 1 "MAX30205MTA+21-0137I_T833-2-M" H 8789 3259 69  0000 L BNN
+F 2 "BodyTempUnit-e7:21-0137I_T833-2-M" H 8200 2900 50  0001 C CNN
+F 3 "" H 8200 2900 50  0001 C CNN
+	1    8200 2900
+	1    0    0    -1
+$EndComp
+Wire Wire Line
+	9700 3100 9800 3100
+Wire Wire Line
+	9800 3100 9800 3000
+Wire Wire Line
+	9700 2900 9800 2900
+Connection ~ 9800 2900
+Wire Wire Line
+	9800 2900 9800 2750
+Wire Wire Line
+	9700 3000 9800 3000
+Connection ~ 9800 3000
+Wire Wire Line
+	9800 3000 9800 2900
+$Comp
+L BodyTempUnit-e7-eagle-import:VCC #SUPPLY06
+U 1 1 A7CD5EB6
+P 8000 2400
+F 0 "#SUPPLY06" H 8000 2400 50  0001 C CNN
+F 1 "VCC" H 7960 2540 59  0000 L BNN
+F 2 "" H 8000 2400 50  0001 C CNN
+F 3 "" H 8000 2400 50  0001 C CNN
+	1    8000 2400
+	1    0    0    -1
+$EndComp
+$Comp
+L BodyTempUnit-e7-eagle-import:VCC #SUPPLY0104
+U 1 1 5D1C5C95
+P 9800 2750
+F 0 "#SUPPLY0104" H 9800 2750 50  0001 C CNN
+F 1 "VCC" H 9760 2890 59  0000 L BNN
+F 2 "" H 9800 2750 50  0001 C CNN
+F 3 "" H 9800 2750 50  0001 C CNN
+	1    9800 2750
+	1    0    0    -1
+$EndComp
+Connection ~ 8000 900
+$Comp
+L Connector_Generic:Conn_01x05 J1
+U 1 1 5D20A11B
+P 1200 1000
+F 0 "J1" H 1118 575 50  0000 C CNN
+F 1 "CONN_IN" H 1118 666 50  0000 C CNN
+F 2 "Connector_Molex:Molex_PicoBlade_53261-0571_1x05-1MP_P1.25mm_Horizontal" H 1200 1000 50  0001 C CNN
+F 3 "~" H 1200 1000 50  0001 C CNN
+	1    1200 1000
+	-1   0    0    1
+$EndComp
+$Comp
+L Connector_Generic:Conn_01x05 J2
+U 1 1 5D20BB11
+P 1200 1700
+F 0 "J2" H 1118 1275 50  0000 C CNN
+F 1 "CONN_OUT" H 1118 1366 50  0000 C CNN
+F 2 "Connector_Molex:Molex_PicoBlade_53261-0571_1x05-1MP_P1.25mm_Horizontal" H 1200 1700 50  0001 C CNN
+F 3 "~" H 1200 1700 50  0001 C CNN
+	1    1200 1700
+	-1   0    0    1
+$EndComp
+Wire Wire Line
+	1400 900  1600 900
+Wire Wire Line
+	1400 1000 1600 1000
+Wire Wire Line
+	1400 1100 1600 1100
+Wire Wire Line
+	1400 800  2150 800
+Wire Wire Line
+	1400 1600 1600 1600
+Wire Wire Line
+	1400 1800 1600 1800
+Wire Wire Line
+	1400 1700 1600 1700
+Wire Wire Line
+	1400 1900 2150 1900
+Text Label 1600 900  0    50   ~ 0
+SIG_IN
+Text Label 1600 1800 0    50   ~ 0
+SIG_OUT
+Wire Wire Line
+	1400 1200 1500 1200
+Wire Wire Line
+	1500 1200 1500 1500
+Wire Wire Line
+	1500 1500 1400 1500
+Wire Wire Line
+	1500 1500 1500 2100
+Connection ~ 1500 1500
+Wire Wire Line
+	4300 5000 4500 5000
+Text Label 4500 5000 0    50   ~ 0
+SIG_OUT
+Wire Wire Line
+	4300 5300 5000 5300
+Wire Wire Line
+	5000 5300 5000 5100
+Wire Wire Line
+	5000 5100 5100 5100
+NoConn ~ 4300 5100
 $EndSCHEMATC

Commit message: version sent to production
Parts:
- added TP1, TP2, TP3, TP4, TP5, TP6, TP7: TestPoint, TestPoint:TestPoint_Pad_D1.0mm, symbol Connector:TestPoint
- C4: footprint BodyTempUnit-e7:C0603K -> Capacitor_SMD:C_0402_1005Metric
- R4: footprint BodyTempUnit-e7:R0603 -> Resistor_SMD:R_0402_1005Metric
Connections:
- net LSM_INT1: now also TP4.1
- net LSM_INT2: now also TP5.1
- net RS485_DE: now also TP3.1
- net U1_OS: now also TP6.1
- net VIN: now also TP1.1
- net at C9.1, U3.5 (VOUT): now also TP2.1
Changed lines of the file:
@@
 	8300 3000 8000 3000
 Wire Wire Line
-	8000 3000 7800 3000
+	8000 3000 7850 3000
 Wire Wire Line
 	8000 3000 8000 2800
@@
 Connection ~ 8000 3000
 Wire Wire Line
-	8500 5300 7900 5300
+	8500 5300 8000 5300
 Text Label 7900 5300 2    50   ~ 0
 LSM_INT1
@@
 LSM_INT1
 Wire Wire Line
-	9500 5500 10000 5500
+	9500 5500 9800 5500
 Text Label 10000 5500 0    50   ~ 0
 LSM_INT2
@@
 F 0 "C4" H 8060 3815 59  0000 L BNN
 F 1 "0.1uF" H 8060 3615 59  0000 L BNN
-F 2 "BodyTempUnit-e7:C0603K" H 8000 3800 50  0001 C CNN
+F 2 "Capacitor_SMD:C_0402_1005Metric" H 8000 3800 50  0001 C CNN
 F 3 "" H 8000 3800 50  0001 C CNN
 	1    8000 3800
@@
 F 0 "R4" H 7850 2659 59  0000 L BNN
 F 1 "R-EU_R0603" H 7850 2470 59  0000 L BNN
-F 2 "BodyTempUnit-e7:R0603" H 8000 2600 50  0001 C CNN
+F 2 "Resistor_SMD:R_0402_1005Metric" H 8000 2600 50  0001 C CNN
 F 3 "" H 8000 2600 50  0001 C CNN
 	1    8000 2600
@@
 	5000 5100 5100 5100
 NoConn ~ 4300 5100
+$Comp
+L Connector:TestPoint TP4
+U 1 1 5D02B287
+P 8000 5300
+F 0 "TP4" H 8058 5418 50  0000 L CNN
+F 1 "TestPoint" H 8058 5327 50  0000 L CNN
+F 2 "TestPoint:TestPoint_Pad_D1.0mm" H 8200 5300 50  0001 C CNN
+F 3 "~" H 8200 5300 50  0001 C CNN
+	1    8000 5300
+	1    0    0    -1
+$EndComp
+Connection ~ 8000 5300
+Wire Wire Line
+	8000 5300 7900 5300
+$Comp
+L Connector:TestPoint TP5
+U 1 1 5D03A148
+P 9800 5500
+F 0 "TP5" H 9858 5618 50  0000 L CNN
+F 1 "TestPoint" H 9858 5527 50  0000 L CNN
+F 2 "TestPoint:TestPoint_Pad_D1.0mm" H 10000 5500 50  0001 C CNN
+F 3 "~" H 10000 5500 50  0001 C CNN
+	1    9800 5500
+	1    0    0    -1
+$EndComp
+Connection ~ 9800 5500
+Wire Wire Line
+	9800 5500 10000 5500
+$Comp
+L Connector:TestPoint TP1
+U 1 1 5D045BEB
+P 2150 800
+F 0 "TP1" H 2208 918 50  0000 L CNN
+F 1 "TestPoint" H 2208 827 50  0000 L CNN
+F 2 "TestPoint:TestPoint_Pad_D1.0mm" H 2350 800 50  0001 C CNN
+F 3 "~" H 2350 800 50  0001 C CNN
+	1    2150 800
+	1    0    0    -1
+$EndComp
+$Comp
+L Connector:TestPoint TP2
+U 1 1 5D048113
+P 4400 1200
+F 0 "TP2" V 4354 1388 50  0000 L CNN
+F 1 "TestPoint" V 4445 1388 50  0000 L CNN
+F 2 "TestPoint:TestPoint_Pad_D1.0mm" H 4600 1200 50  0001 C CNN
+F 3 "~" H 4600 1200 50  0001 C CNN
+	1    4400 1200
+	0    1    1    0
+$EndComp
+Connection ~ 8400 900
+$Comp
+L Connector:TestPoint TP3
+U 1 1 5D061687
+P 6950 1250
+F 0 "TP3" H 7008 1368 50  0000 L CNN
+F 1 "TestPoint" H 7008 1277 50  0000 L CNN
+F 2 "TestPoint:TestPoint_Pad_D1.0mm" H 7150 1250 50  0001 C CNN
+F 3 "~" H 7150 1250 50  0001 C CNN
+	1    6950 1250
+	1    0    0    -1
+$EndComp
+Connection ~ 6950 1250
+$Comp
+L Connector:TestPoint TP6
+U 1 1 5D07F1DE
+P 7850 3000
+F 0 "TP6" H 7908 3118 50  0000 L CNN
+F 1 "TestPoint" H 7908 3027 50  0000 L CNN
+F 2 "TestPoint:TestPoint_Pad_D1.0mm" H 8050 3000 50  0001 C CNN
+F 3 "~" H 8050 3000 50  0001 C CNN
+	1    7850 3000
+	1    0    0    -1
+$EndComp
+Connection ~ 7850 3000
+Wire Wire Line
+	7850 3000 7800 3000
+$Comp
+L Connector:TestPoint TP7
+U 1 1 5D12AA2D
+P 6650 7350
+F 0 "TP7" V 6604 7538 50  0000 L CNN
+F 1 "TestPoint" V 6695 7538 50  0000 L CNN
+F 2 "TestPoint:TestPoint_Pad_D1.0mm" H 6850 7350 50  0001 C CNN
+F 3 "~" H 6850 7350 50  0001 C CNN
+	1    6650 7350
+	0    1    1    0
+$EndComp
+Connection ~ 6650 7350
 $EndSCHEMATC
